File: KiCad/Micro.kicad_sch (KiCad schematic)
At the start: 33 parts, among them J1 Conn_01x02, J1 DE9_Pins, J2 DE9_Pins, J3 Conn_01x05, SW1 SW_Push, U1 MCP4725xxx-xCH, U2 MCP2562-E-SN, U3 MAX3232, U3 PIC24HJ128GP502, Y1 Crystal

Commit message: Totes les footprints seleccionades, part de potencia, placement realitzat
Parts:
- C1, C2, C5, C6, C7, C8, C9: footprint (none) -> Capacitor_SMD:C_1206_3216Metric
- C10: renamed from C5; footprint (none) -> Capacitor_SMD:C_1206_3216Metric
- C11: renamed from C6; footprint (none) -> Capacitor_SMD:C_1206_3216Metric
- C12: renamed from C2; footprint (none) -> Capacitor_SMD:C_1206_3216Metric
- C13: renamed from C7; footprint (none) -> Capacitor_SMD:C_1206_3216Metric
- C14: renamed from C1; footprint (none) -> Capacitor_Tantalum_SMD:CP_EIA-3528-12_Kemet-T
- C3, C4: footprint (none) -> Capacitor_SMD:C_0805_2012Metric
- D1: footprint (none) -> LED_SMD:LED_0805_2012Metric
- FB1, R1, R4: footprint (none) -> Resistor_SMD:R_1206_3216Metric
- J1, J2: footprint (none) -> Connector_Dsub:DSUB-9_Pins_Horizontal_P2.77x2.84mm_EdgePinOffset4.94mm_Housed_MountingHolesOffset4.94mm
- J3: footprint (none) -> Connector_PinHeader_2.54mm:PinHeader_1x05_P2.54mm_Vertical
- J5: renamed from J1; footprint (none) -> Connector_PinHeader_2.54mm:PinHeader_1x02_P2.54mm_Vertical
- R2: renamed from R1; footprint (none) -> Resistor_SMD:R_1206_3216Metric
- R3: renamed from R2; footprint (none) -> Resistor_SMD:R_1206_3216Metric
- R5: renamed from R6; footprint (none) -> Resistor_SMD:R_1206_3216Metric
- R6: renamed from R5; footprint (none) -> Resistor_SMD:R_1206_3216Metric
- R7: renamed from R3; footprint (none) -> Resistor_SMD:R_1206_3216Metric
- SW1: footprint (none) -> Button_Switch_SMD:SW_Push_SPST_NO_Alps_SKRK
- U3: footprint (none) -> Package_SO:SOIC-16_3.9x9.9mm_P1.27mm
- U4: renamed from U3; footprint (none) -> Package_SO:SOIC-28W_7.5x17.9mm_P1.27mm
- renumbered U1 to U5

Commit message: PnR Final versió 1
Connections:
- net CAN_ L is gone; now on net CAN_L: R1.2, U2.6 (CANL)
- net Sortida_RL is gone; now on net 3v3: C2.2, U2.5 (Vio)
- net sortida_RL is gone; now on net 3v3: J3.2 (Pin_2)
Changed lines of the file:
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@@
 		)
 	)
-	(global_label "CAN_ L"
+	(global_label "CAN_L"
 		(shape bidirectional)
 		(at 115.57 52.07 0)
@@
 		)
 		(property "Intersheetrefs" "${INTERSHEET_REFS}"
-			(at 126.3189 52.07 0)
+			(at 125.3513 52.07 0)
 			(effects
 				(font
@@
 		)
 	)
-	(global_label "sortida_RL"
+	(global_label "3v3"
 		(shape output)
 		(at 193.04 49.53 0)
@@
 		)
 		(property "Intersheetrefs" "${INTERSHEET_REFS}"
-			(at 205.8827 49.53 0)
+			(at 199.4118 49.53 0)
 			(effects
 				(font
@@
 		)
 	)
-	(global_label "Sortida_RL"
+	(global_label "3v3"
 		(shape input)
 		(at 62.23 46.99 180)
@@
 		)
 		(property "Intersheetrefs" "${INTERSHEET_REFS}"
-			(at 49.2059 46.99 0)
+			(at 55.8582 46.99 0)
 			(effects
 				(font
@@
 			(project "Micro"
 				(path "/76eb2563-2429-4e39-bcea-6a503034af3e"
-					(reference "C?")
+					(reference "C3")
 					(unit 1)
 				)
@@
 			(project "Micro"
 				(path "/76eb2563-2429-4e39-bcea-6a503034af3e"
-					(reference "#PWR?")
+					(reference "#PWR016")
 					(unit 1)
 				)
@@
 			(project "Micro"
 				(path "/76eb2563-2429-4e39-bcea-6a503034af3e"
-					(reference "#PWR?")
+					(reference "#PWR013")
 					(unit 1)
 				)
@@
 			(project "Micro"
 				(path "/76eb2563-2429-4e39-bcea-6a503034af3e"
-					(reference "C?")
+					(reference "C8")
 					(unit 1)
 				)
@@
 			(project "Micro"
 				(path "/76eb2563-2429-4e39-bcea-6a503034af3e"
-					(reference "C?")
+					(reference "C12")
 					(unit 1)
 				)
@@
 			(project "Micro"
 				(path "/76eb2563-2429-4e39-bcea-6a503034af3e"
-					(reference "#PWR?")
+					(reference "#PWR010")
 					(unit 1)
 				)
@@
 			(project "Micro"
 				(path "/76eb2563-2429-4e39-bcea-6a503034af3e"
-					(reference "#PWR?")
+					(reference "#PWR015")
 					(unit 1)
 				)
@@
 			(project "Micro"
 				(path "/76eb2563-2429-4e39-bcea-6a503034af3e"
-					(reference "#PWR?")
+					(reference "#PWR017")
 					(unit 1)
 				)
@@
 			(project "Micro"
 				(path "/76eb2563-2429-4e39-bcea-6a503034af3e"
-					(reference "#PWR?")
+					(reference "#PWR011")
 					(unit 1)
 				)
@@
 			(project "Micro"
 				(path "/76eb2563-2429-4e39-bcea-6a503034af3e"
-					(reference "#PWR?")
+					(reference "#PWR014")
 					(unit 1)
 				)
@@
 			(project "Micro"
 				(path "/76eb2563-2429-4e39-bcea-6a503034af3e"
-					(reference "J?")
+					(reference "J2")
 					(unit 1)
 				)
@@
 			(project "Micro"
 				(path "/76eb2563-2429-4e39-bcea-6a503034af3e"
-					(reference "C?")
+					(reference "C11")
 					(unit 1)
 				)
@@
 			(project "Micro"
 				(path "/76eb2563-2429-4e39-bcea-6a503034af3e"
-					(reference "C?")
+					(reference "C9")
 					(unit 1)
 				)
@@
 			(project "Micro"
 				(path "/76eb2563-2429-4e39-bcea-6a503034af3e"
-					(reference "J?")
+					(reference "J3")
 					(unit 1)
 				)
@@
 			(project "Micro"
 				(path "/76eb2563-2429-4e39-bcea-6a503034af3e"
-					(reference "C?")
+					(reference "C4")
 					(unit 1)
 				)
@@
 			(project "Micro"
 				(path "/76eb2563-2429-4e39-bcea-6a503034af3e"
-					(reference "C?")
+					(reference "C10")
 					(unit 1)
 				)
@@
 			(project "Micro"
 				(path "/76eb2563-2429-4e39-bcea-6a503034af3e"
-					(reference "#PWR?")
+					(reference "#PWR018")
 					(unit 1)
 				)
@@
 			(project "Micro"
 				(path "/76eb2563-2429-4e39-bcea-6a503034af3e"
-					(reference "U?")
+					(reference "U4")
 					(unit 1)
 				)
@@
 			(project "Micro"
 				(path "/76eb2563-2429-4e39-bcea-6a503034af3e"
-					(reference "C?")
+					(reference "C13")
 					(unit 1)
 				)
@@
 			(project "Micro"
 				(path "/76eb2563-2429-4e39-bcea-6a503034af3e"
-					(reference "Y?")
+					(reference "Y1")
 					(unit 1)
 				)
@@
 			(project "Micro"
 				(path "/76eb2563-2429-4e39-bcea-6a503034af3e"
-					(reference "C?")
+					(reference "C14")
 					(unit 1)
 				)
@@
 			(project "Micro"
 				(path "/76eb2563-2429-4e39-bcea-6a503034af3e"
-					(reference "R?")
+					(reference "R7")
 					(unit 1)
 				)
@@
 			(project "Micro"
 				(path "/76eb2563-2429-4e39-bcea-6a503034af3e"
-					(reference "#PWR?")
+					(reference "#PWR012")
 					(unit 1)
 				)
@@
 			(project "Micro"
 				(path "/76eb2563-2429-4e39-bcea-6a503034af3e"
-					(reference "U?")
+					(reference "U2")
 					(unit 1)
 				)
@@
 			(project "Micro"
 				(path "/76eb2563-2429-4e39-bcea-6a503034af3e"
-					(reference "J?")
+					(reference "J4")
 					(unit 1)
 				)
