File: KiCad/Micro.kicad_sch (KiCad schematic)
At the start: 33 parts, among them J1 DE9_Pins, J2 DE9_Pins, J3 Conn_01x05, J5 Conn_01x02, SW1 SW_Push, U2 MCP2562-E-SN, U3 MAX3232, U4 PIC24HJ128GP502, U5 MCP4725xxx-xCH, Y1 Crystal

Commit message: pnr editat
Parts:
- J3: footprint Connector_PinHeader_2.54mm:PinHeader_1x05_P2.54mm_Vertical -> TerminalBlock_TE-Connectivity:TerminalBlock_TE_282834-5_1x05_P2.54mm_Horizontal
- J5: footprint Connector_PinHeader_2.54mm:PinHeader_1x02_P2.54mm_Vertical -> TerminalBlock_TE-Connectivity:TerminalBlock_TE_282834-2_1x02_P2.54mm_Horizontal
Changed lines of the file:
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@@
 			)
 		)
-		(property "Footprint" "Connector_PinHeader_2.54mm:PinHeader_1x02_P2.54mm_Vertical"
+		(property "Footprint" "TerminalBlock_TE-Connectivity:TerminalBlock_TE_282834-2_1x02_P2.54mm_Horizontal"
 			(at 182.88 138.43 0)
 			(effects
@@
 			)
 		)
-		(property "Footprint" "Connector_PinHeader_2.54mm:PinHeader_1x05_P2.54mm_Vertical"
+		(property "Footprint" "TerminalBlock_TE-Connectivity:TerminalBlock_TE_282834-5_1x05_P2.54mm_Horizontal"
 			(at 187.96 46.99 0)
 			(effects

Commit message: -
Connections:
- net 3v3: no longer U2.5 (Vio)
- net CAN_H renamed CAN_H_+
- net CAN_L renamed CAN_L_-
Other:
- moved on the sheet: C1, C2, J1, R1, U2

Commit message: -
Connections:
- net CAN_H_+ renamed USB_H_P
- net CAN_L_- renamed USB_L_N
Changed lines of the file:
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@@
 		)
 	)
-	(global_label "CAN_L_-"
+	(global_label "USB_L_N"
 		(shape bidirectional)
 		(at 30.48 45.72 0)
@@
 		)
 		(property "Intersheetrefs" "${INTERSHEET_REFS}"
-			(at 42.8013 45.72 0)
+			(at 42.6803 45.72 0)
 			(effects
 				(font
@@
 		)
 	)
-	(global_label "CAN_H_+"
+	(global_label "USB_H_P"
 		(shape bidirectional)
 		(at 30.48 48.26 0)
@@
 		)
 		(property "Intersheetrefs" "${INTERSHEET_REFS}"
-			(at 43.1037 48.26 0)
+			(at 42.9222 48.26 0)
 			(effects
 				(font
@@
 		)
 	)
-	(global_label "CAN_L_-"
+	(global_label "USB_L_N"
 		(shape bidirectional)
 		(at 68.834 40.894 180)
@@
 		)
 		(property "Intersheetrefs" "${INTERSHEET_REFS}"
-			(at 56.5127 40.894 0)
+			(at 56.6337 40.894 0)
 			(effects
 				(font
@@
 		)
 	)
-	(global_label "CAN_H_+"
+	(global_label "USB_H_P"
 		(shape bidirectional)
 		(at 68.834 57.404 180)
@@
 		)
 		(property "Intersheetrefs" "${INTERSHEET_REFS}"
-			(at 56.2103 57.404 0)
-			(effects
-				(font
+			(at 56.3918 57.404 0)
+			(effects
+				(font
