File: KiCad/Combustible_projecte.kicad_pcb (KiCad board)
At the start: 2 copper layers, 103.1 x 69.4 mm, 60 parts, among them J1 DE9_Pins, J2 DE9_Pins, J20 Conn_01x02, J3 Conn_01x05, J4 Conn_01x02, J5 Conn_01x02, J6 Conn_01x02, Q1 2N7002, Q2 2N7002, SW1 SW_Push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

Commit message: millora pcb
Routing:
- net Net-(U4-/MCLR): track 3.89 -> 21.3 mm
Changed lines of the file:
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@@
+	)
+	(segment
+		(start 98.977 54.1605)
+		(end 116.5605 54.1605)
+		(width 0.2)
+		(layer "F.Cu")
+		(net 46)
 	)
 	(segment
@@
 	)
 	(segment
-		(start 115.861 53.461)
+		(start 116.5605 54.1605)
 		(end 118.03 55.63)
 		(width 0.2)
 		(layer "F.Cu")
+		(net 46)
+	)
+	(segment
+		(start 98.4 54.7375)
+		(end 98.977 54.1605)
+		(width 0.2)
+		(layer "F.Cu")

Commit message: -
Connections:
- net CAN_H renamed CAN_H_+
- net CAN_L renamed CAN_L_-
- C2 pad 1: GND -> unconnected-(C2-Pad1)
- U2 pad 5: 3v3 -> unconnected-(U2-Vio-Pad5)
Routing:
- net CAN_L_-: track 55.2 -> 3.97 mm
- net CAN_H_+: track 53.3 -> 3.82 mm

Commit message: millora vies gnd
Routing:
- net GND: track 36.7 -> 12.7 mm, vias 88 -> 91

Commit message: -
Connections:
- net CAN_H_+ renamed USB_H_P
- net CAN_L_- renamed USB_L_N
- C2 pad 1: unconnected-(C2-Pad1) -> GND
Changed lines of the file:
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@@
 	(net 64 "unconnected-(U4-RB5-Pad14)")
 	(net 65 "unconnected-(U5-A0-Pad6)")
-	(net 66 "CAN_H_+")
-	(net 67 "CAN_L_-")
-	(net 68 "unconnected-(C2-Pad1)")
-	(net 69 "unconnected-(U2-Vio-Pad5)")
+	(net 66 "USB_H_P")
+	(net 67 "USB_L_N")
+	(net 68 "unconnected-(U2-Vio-Pad5)")
 	(footprint "MountingHole:MountingHole_2.1mm"
 		(layer "F.Cu")
@@
 			(layers "F.Cu" "F.Mask" "F.Paste")
 			(roundrect_rratio 0.217391)
-			(net 68 "unconnected-(C2-Pad1)")
+			(net 2 "GND")
 			(pintype "passive")
 		)
@@
 			(layers "F.Cu" "F.Mask" "F.Paste")
 			(roundrect_rratio 0.25)
-			(net 69 "unconnected-(U2-Vio-Pad5)")
+			(net 68 "unconnected-(U2-Vio-Pad5)")
 			(pinfunction "Vio")
 			(pintype "power_in")
@@
 			(layers "F.Cu" "F.Mask" "F.Paste")
 			(roundrect_rratio 0.25)
-			(net 67 "CAN_L_-")
+			(net 67 "USB_L_N")
 			(pinfunction "CANL")
 			(pintype "bidirectional")
@@
 			(layers "F.Cu" "F.Mask" "F.Paste")
 			(roundrect_rratio 0.25)
-			(net 66 "CAN_H_+")
+			(net 66 "USB_H_P")
 			(pinfunction "CANH")
 			(pintype "bidirectional")
@@
 			(layers "F.Cu" "F.Mask" "F.Paste")
 			(roundrect_rratio 0.222222)
-			(net 66 "CAN_H_+")
+			(net 66 "USB_H_P")
 			(pintype "passive")
 		)
@@
 			(layers "F.Cu" "F.Mask" "F.Paste")
 			(roundrect_rratio 0.222222)
-			(net 67 "CAN_L_-")
+			(net 67 "USB_L_N")
 			(pintype "passive")
 		)
@@
 			(layers "*.Cu" "*.Mask")
 			(remove_unused_layers no)
-			(net 67 "CAN_L_-")
+			(net 67 "USB_L_N")
 			(pinfunction "2")
 			(pintype "passive")
@@
 			(layers "*.Cu" "*.Mask")
 			(remove_unused_layers no)
-			(net 66 "CAN_H_+")
+			(net 66 "USB_H_P")
 			(pinfunction "7")
 			(pintype "passive")
