File: KiCad/analog.kicad_sch (KiCad schematic)
At the start: 23 parts, among them J20 Conn_01x02, J4 Conn_01x02, J6 Conn_01x02, Q1 2N7002, Q2 2N7002, U1 LM1117T-3.3, U20 LM2596T-5

Commit message: pnr editat
Parts:
- J20, J4, J6: footprint Connector_PinHeader_2.54mm:PinHeader_1x02_P2.54mm_Vertical -> TerminalBlock_TE-Connectivity:TerminalBlock_TE_282834-2_1x02_P2.54mm_Horizontal
Changed lines of the file:
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@@
 			)
 		)
-		(property "Footprint" "Connector_PinHeader_2.54mm:PinHeader_1x02_P2.54mm_Vertical"
+		(property "Footprint" "TerminalBlock_TE-Connectivity:TerminalBlock_TE_282834-2_1x02_P2.54mm_Horizontal"
 			(at 147.32 115.57 0)
 			(effects
@@
 			)
 		)
-		(property "Footprint" "Connector_PinHeader_2.54mm:PinHeader_1x02_P2.54mm_Vertical"
+		(property "Footprint" "TerminalBlock_TE-Connectivity:TerminalBlock_TE_282834-2_1x02_P2.54mm_Horizontal"
 			(at 252.73 114.3 0)
 			(effects
@@
 			)
 		)
-		(property "Footprint" "Connector_PinHeader_2.54mm:PinHeader_1x02_P2.54mm_Vertical"
+		(property "Footprint" "TerminalBlock_TE-Connectivity:TerminalBlock_TE_282834-2_1x02_P2.54mm_Horizontal"
 			(at 24.13 54.61 0)
 			(effects

Commit message: Ultims canvis i completat el README
Other:
- moved on the sheet: J6
Changed lines of the file:
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@@
 	)
 	(junction
-		(at 33.02 49.53)
+		(at 49.53 49.53)
 		(diameter 0)
 		(color 0 0 0 0)
@@
 	(wire
 		(pts
-			(xy 33.02 49.53) (xy 54.61 49.53)
+			(xy 49.53 49.53) (xy 54.61 49.53)
 		)
 		(stroke
@@
 	(wire
 		(pts
-			(xy 31.75 54.61) (xy 31.75 57.15)
+			(xy 48.26 54.61) (xy 48.26 57.15)
 		)
 		(stroke
@@
 	(wire
 		(pts
-			(xy 33.02 49.53) (xy 33.02 52.07)
+			(xy 49.53 49.53) (xy 49.53 52.07)
 		)
 		(stroke
@@
 	(wire
 		(pts
-			(xy 33.02 48.26) (xy 31.75 48.26)
+			(xy 49.53 48.26) (xy 48.26 48.26)
 		)
 		(stroke
@@
 	(wire
 		(pts
-			(xy 33.02 52.07) (xy 29.21 52.07)
+			(xy 49.53 52.07) (xy 45.72 52.07)
 		)
 		(stroke
@@
 	(wire
 		(pts
-			(xy 29.21 54.61) (xy 31.75 54.61)
+			(xy 45.72 54.61) (xy 48.26 54.61)
 		)
 		(stroke
@@
 	(wire
 		(pts
-			(xy 33.02 48.26) (xy 33.02 49.53)
+			(xy 49.53 48.26) (xy 49.53 49.53)
 		)
 		(stroke
@@
 	(global_label "VBAT"
 		(shape output)
-		(at 31.75 48.26 90)
+		(at 48.26 48.26 90)
 		(fields_autoplaced yes)
 		(effects
@@
 		)
 		(property "Intersheetrefs" "${INTERSHEET_REFS}"
-			(at 31.75 40.86 90)
+			(at 48.26 40.86 90)
 			(effects
 				(font
@@
 		(on_board yes)
 		(dnp no)
-		(fields_autoplaced yes)
 		(property "Reference" "C16"
 			(at 153.67 59.0549 0)
@@
 	(symbol
 		(lib_id "Connector_Generic:Conn_01x02")
-		(at 24.13 54.61 180)
+		(at 40.64 54.61 180)
 		(unit 1)
 		(exclude_from_sim no)
@@
 		(fields_autoplaced yes)
 		(property "Reference" "J6"
-			(at 24.13 45.72 0)
+			(at 40.64 45.72 0)
 			(effects
 				(font
@@
 		)
 		(property "Value" "Conn_01x02"
-			(at 24.13 48.26 0)
+			(at 40.64 48.26 0)
 			(effects
 				(font
@@
 		)
 		(property "Footprint" "TerminalBlock_TE-Connectivity:TerminalBlock_TE_282834-2_1x02_P2.54mm_Horizontal"
-			(at 24.13 54.61 0)
+			(at 40.64 54.61 0)
 			(effects
 				(font
@@
 		)
 		(property "Datasheet" "~"
-			(at 24.13 54.61 0)
+			(at 40.64 54.61 0)
 			(effects
 				(font
@@
 		)
 		(property "Description" "Generic connector, single row, 01x02, script generated (kicad-library-utils/schlib/autogen/connector/)"
-			(at 24.13 54.61 0)
+			(at 40.64 54.61 0)
 			(effects
 				(font
@@
 	(symbol
 		(lib_id "power:GND")
-		(at 31.75 57.15 0)
+		(at 48.26 57.15 0)
 		(unit 1)
 		(exclude_from_sim no)
@@
 		(fields_autoplaced yes)
 		(property "Reference" "#PWR0112"
-			(at 31.75 63.5 0)
+			(at 48.26 63.5 0)
 			(effects
 				(font
@@
 		)
 		(property "Value" "GND"
-			(at 31.75 62.23 0)
+			(at 48.26 62.23 0)
 			(effects
 				(font
@@
 		)
 		(property "Footprint" ""
-			(at 31.75 57.15 0)
+			(at 48.26 57.15 0)
 			(effects
 				(font
@@
 		)
 		(property "Datasheet" ""
-			(at 31.75 57.15 0)
+			(at 48.26 57.15 0)
 			(effects
 				(font
@@
 		)
 		(property "Description" "Power symbol creates a global label with name \"GND\" , ground"
-			(at 31.75 57.15 0)
+			(at 48.26 57.15 0)
 			(effects
 				(font
